File: battery_3s_18650.sch (KiCad schematic (older format))
At the start: 6 parts, among them U2 MCQ4407

Commit message: 4.1uH antenna project done. Antenna was added to project via bitmap.
Parts:
- BT1, BT2, BT3: footprint NFC_hatch_tmp:18650_holder_SMD -> NFC_hatch_tmp:18650_holder_SMD_65mm
Changed lines of the file:
@@
 F 0 "BT3" V 4250 3900 50  0000 L CNN
 F 1 "18650" V 4350 3850 50  0000 L CNN
-F 2 "NFC_hatch_tmp:18650_holder_SMD" V 4500 3960 50  0001 C CNN
+F 2 "NFC_hatch_tmp:18650_holder_SMD_65mm" V 4500 3960 50  0001 C CNN
 F 3 "~" V 4500 3960 50  0001 C CNN
 	1    4500 3900
-	1    0    0    -1
-$EndComp
-$Comp
-L Device:Battery_Cell BT2
-U 1 1 5F434D15
-P 4500 3500
-F 0 "BT2" V 4250 3500 50  0000 L CNN
-F 1 "18650" V 4350 3450 50  0000 L CNN
-F 2 "NFC_hatch_tmp:18650_holder_SMD" V 4500 3560 50  0001 C CNN
-F 3 "~" V 4500 3560 50  0001 C CNN
-	1    4500 3500
 	1    0    0    -1
 $EndComp
@@
 F 0 "BT1" V 4250 3100 50  0000 L CNN
 F 1 "18650" V 4350 3050 50  0000 L CNN
-F 2 "NFC_hatch_tmp:18650_holder_SMD" V 4500 3160 50  0001 C CNN
+F 2 "NFC_hatch_tmp:18650_holder_SMD_65mm" V 4500 3160 50  0001 C CNN
 F 3 "~" V 4500 3160 50  0001 C CNN
 	1    4500 3100
@@
 	5800 3450 5800 3350
 Connection ~ 5800 3350
+$Comp
+L Device:Battery_Cell BT2
+U 1 1 5F434D15
+P 4500 3500
+F 0 "BT2" V 4250 3500 50  0000 L CNN
+F 1 "18650" V 4350 3450 50  0000 L CNN
+F 2 "NFC_hatch_tmp:18650_holder_SMD_65mm" V 4500 3560 50  0001 C CNN
+F 3 "~" V 4500 3560 50  0001 C CNN
+	1    4500 3500
+	1    0    0    -1
+$EndComp
 $EndSCHEMATC

Commit message: 4.32uH Antenna board done!
Other:
- note removed: "1210"
Changed lines of the file:
@@
 	4800 3050 4800 2950
 Text Notes 5950 3750 0    50   ~ 0
-1210
+0603
 Text Notes 5300 3750 0    50   ~ 0
 0603
